File: Scheatic_Integrated_ACG_separate_v2_by_L.Battisti/Integrated_ACG_separate_v2.kicad_pcb (KiCad board)
At the start: 4 copper layers, 64 x 24.5 mm, 33 parts, among them IC1 ATMEGA328PB-MUR, J1 Conn_01x04_Pin, J2 FLASH, J3 84952-5, U1 TLC5947RHB, U2 TJA1028TK/5V0/20/J, Y1 Crystal_GND24

Commit message: Add new LED functions and update charging effect
Parts:
- moved R3 2.90 mm to (216.8, 154.2), turned to 180 degrees
- moved C2 1.64 mm to (216.8, 136.5)
- moved R2 1.45 mm to (217.5, 133.1)
Routing:
- net /uController/RST: track 49.1 -> 46.2 mm
- net +5V: track 14.3 -> 12.6 mm
- net GND: track 33.6 -> 32.0 mm
- net /uController/LIN: track 16.7 -> 17.3 mm
Other:
- outline, holes or cut-outs redrawn
