File: Scheatic_Integrated_ACG_separate_v2_by_L.Battisti/LED_Driver.kicad_sch (KiCad schematic)
At the start: 19 parts, among them U1 TLC5947RHB

Commit message: Add new LED functions and update charging effect
Parts:
- L1, L2, L3, L4: footprint 00_RA_Library:LRTB GVSG_OSR -> 00_I_Cagol_FootPrint_library:LRTBGVSR4U4VJW8A8BD83S4U7Z
Changed lines of the file:
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@@
 			)
 		)
-		(property "Footprint" "00_RA_Library:LRTB GVSG_OSR"
+		(property "Footprint" "00_I_Cagol_FootPrint_library:LRTBGVSR4U4VJW8A8BD83S4U7Z"
 			(at 160.02 90.17 0)
 			(effects
@@
 			)
 		)
-		(property "Footprint" "00_RA_Library:LRTB GVSG_OSR"
+		(property "Footprint" "00_I_Cagol_FootPrint_library:LRTBGVSR4U4VJW8A8BD83S4U7Z"
 			(at 160.02 107.95 0)
 			(effects
@@
 			)
 		)
-		(property "Footprint" "00_RA_Library:LRTB GVSG_OSR"
+		(property "Footprint" "00_I_Cagol_FootPrint_library:LRTBGVSR4U4VJW8A8BD83S4U7Z"
 			(at 160.02 72.39 0)
 			(effects
@@
 			)
 		)
-		(property "Footprint" "00_RA_Library:LRTB GVSG_OSR"
+		(property "Footprint" "00_I_Cagol_FootPrint_library:LRTBGVSR4U4VJW8A8BD83S4U7Z"
 			(at 160.02 54.61 0)
 			(effects
